Commit message: Add MuJoCo simulation data workflow

File: software/lerobot-hei-rebot-lift/examples/hei_rebot_lift/VR_mujoco_ik/mujoco_ik/model/HEI_robot_urdf/urdf/HEI_robot_urdf.urdf (robot description, URDF)
Before this commit: robot HEI_robot_urdf, 32 links, 31 joints
Links:
- added link front_camera_link, mass 0.0159332340793735; collision mesh filename=../meshes/front_camera_link.STL; visual mesh filename=../meshes/front_camera_link.STL
- added link front_camera_optical_frame
- added link left_wrist_camera_link, mass 0.0357371195664808; collision mesh filename=../meshes/left_wrist_camera_link.STL; visual mesh filename=../meshes/left_wrist_camera_link.STL
- added link left_wrist_camera_optical_frame
- added link right_wrist_camera_link, mass 0.0357371195664808; collision mesh filename=../meshes/right_wrist_camera_link.STL; visual mesh filename=../meshes/right_wrist_camera_link.STL
- added link right_wrist_camera_optical_frame
Joints:
- added joint front_camera_joint: type fixed, parent lift_carriage_link, child front_camera_link, origin xyz=0.117677245413621 -0.000399999999995397 0.294449693458613 rpy=2.1816615649929 0 1.57079632679492
- added joint front_camera_optical_joint: type fixed, parent front_camera_link, child front_camera_optical_frame, origin xyz=0 0 0 rpy=0 0 3.14159265358979
- added joint left_wrist_camera_joint: type fixed, parent b_left_link6, child left_wrist_camera_link, origin xyz=0.090466 0 0.060578 rpy=1.8326 0 1.5708
- added joint left_wrist_camera_optical_joint: type fixed, parent left_wrist_camera_link, child left_wrist_camera_optical_frame, origin xyz=0 0 0 rpy=0 0 3.14159265358979
- added joint right_wrist_camera_joint: type fixed, parent a_right_link6, child right_wrist_camera_link, origin xyz=0.090465710248936 0 0.0605783166800833 rpy=1.83259571459404 0 1.5707963267949
- added joint right_wrist_camera_optical_joint: type fixed, parent right_wrist_camera_link, child right_wrist_camera_optical_frame, origin xyz=0 0 0 rpy=0 0 3.14159265358979
